Commit message: change urdf for test
change rpm can change the 0

File: urdf3/xuepen.urdf (robot description, URDF)
Before this commit: robot xuepen_robot, 3 links, 2 joints
Joints:
- joint joint1: axis 1 0 0 -> 0 1 0; limit lower=0.0 upper=0.548 effort=1000.0 velocity=0.5 -> lower=0.0 upper=6.28 effort=6.28 velocity=0.5; origin xyz=0 0 .35 rpy=0 0 0 -> xyz=0 0 .35 rpy=0 1.57 0
